Commit message: path plan v1

File: my_car/my_car/wildbot.urdf (robot description, URDF)
Before this commit: robot wildbot, 8 links, 7 joints
Links:
- added link arm1_link, mass 0.06; collision box size=0.080 0.03 0.03; visual box size=0.080 0.03 0.03
- added link arm2_link, mass 0.06; collision box size=0.065 0.025 0.025; visual box size=0.065 0.025 0.025
- added link finger_base, mass 0.03; collision box size=0.02 0.05 0.02; visual box size=0.02 0.05 0.02
- added link finger_left, mass 0.01; collision mesh filename=mesh/finger_left.stl scale=0.001 0.001 0.001; visual mesh filename=mesh/finger_left.stl scale=0.001 0.001 0.001
- added link finger_right, mass 0.01; collision mesh filename=mesh/finger_right.stl scale=0.001 0.001 0.001; visual mesh filename=mesh/finger_right.stl scale=0.001 0.001 0.001
- added link ir_side_sensor, mass 0.005; collision box size=0.012 0.006 0.006; visual box size=0.012 0.006 0.006
- link safe_box: geometry collision box size=0.003 0.300 0.100; collision box size=0.315 0.003 0.100
Joints:
- added joint arm1_to_arm2_joint: type revolute, parent arm1_link, child arm2_link, origin xyz=0.080 0.0 0.0 rpy=0 0 0, axis 0 1 0
- added joint arm2_to_finger: type fixed, parent arm2_link, child finger_base, origin xyz=0.065 0.0 0.0 rpy=0 0 0
- added joint finger_base_to_finger_left: type revolute, parent finger_base, child finger_left, origin xyz=0.0 0.014 0.0 rpy=0 0 0, axis 0 0 1
- added joint finger_base_to_finger_right: type revolute, parent finger_base, child finger_right, origin xyz=0.0 -0.014 0.0 rpy=0 0 0, axis 0 0 1
- added joint finger_base_to_ir_side_sensor: type fixed, parent finger_base, child ir_side_sensor, origin xyz=0.0 0.035 0.0 rpy=0 0 -0.5
- added joint safe_box_to_arm1_joint: type revolute, parent safe_box, child arm1_link, origin xyz=0.170 0.0 0.026 rpy=0 0 0, axis 0 1 0
- joint safe_box_to_camera: origin xyz=0.105 0.0 0.155 rpy=-1.89 0.0 -1.57 -> xyz=0.005 0.0 0.275 rpy=-1.89 0 -1.57
- joint safe_box_to_lidar: origin xyz=0.050 0.0 0.190 rpy=0 0 0 -> xyz=-0.050 0.0 0.310 rpy=0 0 0

Commit message: 5/23

File: my_car/my_car/wildbot.urdf (robot description, URDF)
Before this commit: robot wildbot, 14 links, 13 joints
Joints:
- joint arm1_to_arm2_joint: limit (none) -> lower=-1.5708 upper=1.5708 effort=10.0 velocity=1.0
- joint finger_base_to_finger_left: limit (none) -> lower=-0.7854 upper=0.7854 effort=2.0 velocity=1.0
- joint finger_base_to_finger_right: limit (none) -> lower=-0.7854 upper=0.7854 effort=2.0 velocity=1.0
- joint safe_box_to_arm1_joint: limit (none) -> lower=-1.5708 upper=1.5708 effort=10.0 velocity=1.0
