Commit message: 000

File: bridge/wildbot.urdf (robot description, URDF)
Before this commit: robot wildbot, 14 links, 13 joints
Links:
- added link camera_link, mass 0.005; visual box size=0.01 0.01 0.01
Joints:
- removed joint safe_box_to_camera
- added joint camera_link_to_camera: type fixed, parent camera_link, child camera, origin xyz=0 0 0 rpy=0 0 0
- added joint safe_box_to_camera_link: type fixed, parent safe_box, child camera_link, origin xyz=0.005 0.0 0.275 rpy=0 0.28 0

File: my_car/my_car/wildbot.urdf (robot description, URDF)
Before this commit: robot wildbot, 14 links, 13 joints
Links:
- added link camera_link, mass 0.005; visual box size=0.01 0.01 0.01
Joints:
- removed joint safe_box_to_camera
- added joint camera_link_to_camera: type fixed, parent camera_link, child camera, origin xyz=0 0 0 rpy=0 0 0
- added joint safe_box_to_camera_link: type fixed, parent safe_box, child camera_link, origin xyz=-0.02 0.0 0.275 rpy=0 0.28 0
- joint safe_box_to_arm1_joint: origin xyz=0.170 0.0 0.026 rpy=0 0 0 -> xyz=0.170 0.0 0.029 rpy=0 0 0
- joint safe_box_to_lidar: origin xyz=-0.050 0.0 0.310 rpy=0 0 0 -> xyz=-0.070 0.0 0.310 rpy=0 0 0
